File: Kicad/thermocouple/thermocouple.kicad_pcb (KiCad board)
At the start: 2 copper layers, 38.5 x 61.5 mm, 19 parts, among them IC1 LM335AZT, J1 Thermocouple, J2 DC_in, J3 Conn_01x10_Socket, U1 AD620, U3 WeMos_S2_mini, U4 TL431LP, U5 LM358

Commit message: Release Update readme Added wifi interface Add wifi UI Calibration Add DAC
Parts:
- removed IC1: LM335AZT, Package_TO_SOT_THT:TO-92L_HandSolder
- removed R1, R4: 10k, Resistor_SMD:R_1206_3216Metric_Pad1.30x1.75mm_HandSolder
- removed R2, R3, R6: R, Resistor_SMD:R_1206_3216Metric_Pad1.30x1.75mm_HandSolder
- removed RV2, RV4, RV5: 1k, Potentiometer_SMD:Potentiometer_Bourns_TC33X_Vertical
- removed U4: TL431LP, Package_TO_SOT_THT:TO-92_HandSolder
- added J4: DHT, Connector_PinHeader_2.54mm:PinHeader_1x03_P2.54mm_Vertical, F.Cu at (74.4, 110.5)
- J1: footprint Connector_PinHeader_2.54mm:PinHeader_1x02_P2.54mm_Vertical -> TerminalBlock:TerminalBlock_MaiXu_MX126-5.0-02P_1x02_P5.00mm
- R5: value R -> 1k
- moved R5 22.8 mm to (87.0, 88.2)
- moved RV1 15.2 mm to (81.8, 101.8)
- moved U1 13.0 mm to (85.4, 105.6)
- moved J2 11.8 mm to (106.5, 93.0)
- moved J1 8.17 mm to (100.2, 105.5), turned to 90 degrees
- moved U5 3.86 mm to (87.3, 80.6), turned to 180 degrees
- moved RV3 2.01 mm to (84.8, 71.0), turned to 180 degrees
Connections:
- J1 pad 2: TC+ -> Ref
- J3 pad 5: LCD_RW -> GND
- U1 pad 3: TC+ -> Ref
- U3 pad 27: unconnected-(U3-DAC_1-Pad27) -> Ref
- U3 pad 7: unconnected-(U3-GPIO12-Pad7) -> DHT
- U5 pad 5: Ref -> (no net)
- U5 pad 6: Net-(U5B--) -> (no net)
- U5 pad 7: ADC1_1 -> (no net)
Routing:
- net GND: track 138.8 -> 11.2 mm
- net Net-(IC1-V+): track 32.1 -> 0.00 mm
- net DC_IN: track 52.7 -> 79.5 mm
- net DHT: track 0.00 -> 26.3 mm
- net ADC1_1: track 24.3 -> 0.00 mm
- net Net-(U5A--): track 40.9 -> 21.5 mm
- net TC+: track 17.0 -> 0.00 mm
- net +3V3: track 27.3 -> 42.2 mm
- net Net-(U5B--): track 13.1 -> 0.00 mm
- net Net-(U4-REF): track 10.8 -> 0.00 mm
- net LCD_RW: track 8.86 -> 0.00 mm
- net TC-: track 20.5 -> 14.4 mm
- net Net-(IC1-ADJ): track 6.00 -> 0.00 mm
- net DIFF: track 15.2 -> 10.8 mm
- net Ref: track 39.1 -> 35.0 mm
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Other:
- board size 38.5 x 61.5 mm -> 37.2 x 52.5 mm
