File: Kicad/thermocouple/thermocouple.kicad_sch (KiCad schematic)
At the start: 19 parts, among them IC1 LM335AZT, J1 Thermocouple, J2 DC_in, J3 Conn_01x10_Socket, U1 AD620, U3 WeMos_S2_mini, U4 TL431LP, U5 LM358

Commit message: TestCircuit DAC configured
Other:
- title: (none) -> Thermocouple
Changed lines of the file:
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@@
 	(generator_version "9.0")
 	(paper "USLetter")
+	(title_block
+		(title "Thermocouple")
+	)
 	(rectangle
 		(start 16.51 16.51)

Commit message: Release Update readme Added wifi interface Add wifi UI Calibration Add DAC
Parts:
- removed IC1: LM335AZT, Package_TO_SOT_THT:TO-92L_HandSolder, symbol LM335AZT:LM335AZT
- removed J1: Thermocouple, Connector_PinHeader_2.54mm:PinHeader_1x02_P2.54mm_Vertical, symbol Connector_Generic:Conn_01x02
- removed R1, R4: 10k, Resistor_SMD:R_1206_3216Metric_Pad1.30x1.75mm_HandSolder, symbol Device:R
- removed R2, R3, R6: R, Resistor_SMD:R_1206_3216Metric_Pad1.30x1.75mm_HandSolder, symbol Device:R
- removed RV2, RV4, RV5: 1k, Potentiometer_SMD:Potentiometer_Bourns_TC33X_Vertical, symbol Device:R_Potentiometer
- removed U4: TL431LP, Package_TO_SOT_THT:TO-92_HandSolder, symbol Reference_Voltage:TL431LP
- removed unit 2 of U5
- added J1: Thermocouple, TerminalBlock:TerminalBlock_MaiXu_MX126-5.0-02P_1x02_P5.00mm, symbol Connector:Screw_Terminal_01x02
- added J4: DHT, Connector_PinHeader_2.54mm:PinHeader_1x03_P2.54mm_Vertical, symbol Connector_Generic:Conn_01x03
- R5: value R -> 1k
Connections:
- net TC+ is gone; now on net Ref: U1.3 (+)
- net +3V3: now also J4.3 (Pin_3)
- net GND: now also J3.5 (Pin_5), J4.2 (Pin_2)
- net LCD_RW: no longer J3.5 (Pin_5)
- net Ref: now also U3.27 (DAC_1), J1.2 (Pin_2)
- net TC-: now also J1.1 (Pin_1)
- net DHT: now reaches U3.7 (GPIO12)
- net DHT: now also J4.1 (Pin_1)
Other:
- note added: "Temperature Reference"
- note removed: "AD620 Virtual Ground (REF)"
- note removed: "El integrado LM355 proporciona 10mV/K lo que a temperatura ambiente es ~3v a los ~57C excede la entrada del ADC, por lo que se calibra con un amplificador operacional subrayendo el voltaje de referencia y amplificando. Aunque la temperatura ambiente no deberia llegar a tales valores, se utiliza como criterio de seguridad y para mejorar la resolucion a la entrada del ADC"
- note removed: "Op Amp Supply"
- note removed: "Temperature Reference Amplification Stage"
- note removed: "Tierra Virtual para el AD620 El uso de un divisor resistivo es inestable en comparacion de un voltaje de referencia"
- moved on the sheet: R5, RV1, RV3, U1, U5A, U5C
